File: TeensyTest/TeensyTest.sch (KiCad schematic (older format))
At the start: 32 parts, among them J2 Conn_01x08_Female, J3 Conn_01x04_Female, P1 USB_C_Plug_USB2.0, SW1 SW_Push, SW2 SW_Push, U1 AP2114H, U2 MK20DX256VLH7, U3 MKL02Z32VFG4, Y1 Crystal_GND24

Commit message: Initial commit
Parts:
- removed J2: Conn_01x08_Female, Connector_PinHeader_2.54mm:PinHeader_1x08_P2.54mm_Vertical, symbol Connector:Conn_01x08_Female
- removed J3: Conn_01x04_Female, Connector_PinHeader_2.54mm:PinHeader_1x04_P2.54mm_Vertical, symbol Connector:Conn_01x04_Female
- removed SW1, SW2: SW_Push, Button_Switch_SMD:SW_SPST_EVQQ2, symbol Switch:SW_Push
- removed U1: AP2114H, Package_TO_SOT_SMD:SOT-223-3_TabPin2, symbol Regulator_Linear:AP1117-33
- added 0.1uF1: C, Capacitor_SMD:C_0603_1608Metric, symbol Device:C
- added C12: 220pF, Capacitor_SMD:C_0603_1608Metric, symbol Device:C
- added C13: 10uF, Capacitor_SMD:C_0805_2012Metric, symbol Device:C_Small
- added C14, C16, C17: 0.1uF, Capacitor_SMD:C_0805_2012Metric, symbol Device:C
- added C15: 0.1uF, Capacitor_SMD:C_0603_1608Metric, symbol Device:C_Small
- added C26: 1nF, Capacitor_SMD:C_0603_1608Metric, symbol Device:C
- added D11: SM24CANB-02HTG, SM24CANB02HTG, symbol SamacSys_Parts:SM24CANB-02HTG
- added D2, D3, D4: D, Diode_SMD:D_SMA, symbol Device:D
- added D5: SMBJ33A, SamacSys_Parts:DIOM5436X244N, symbol SamacSys_Parts:SMBJ33A
- added F2: Fuse, Fuse:Fuse_1812_4532Metric, symbol Device:Fuse
- added H3, H4: MountingHole, MountingHole:MountingHole_3.2mm_M3_DIN965_Pad, symbol Mechanical:MountingHole
- added H5, H6, H7, H8: MountingHole_Pad, MountingHole:MountingHole_3.2mm_M3_DIN965_Pad_TopBottom, symbol Mechanical:MountingHole_Pad
- added IC3: TJA1027T/20,118, SamacSys_Parts:SOIC127P600X175-8N, symbol SamacSys_Parts:TLIN2029DRQ1
- added IC4: LM1117MPX-3.3_NOPB, SamacSys_Parts:SOT230P700X180-4N, symbol SamacSys_Parts:LM1117MPX-3.3_NOPB
- added J1: 431151015826, SamacSys_Parts:431151015826, symbol SamacSys_Parts:431151015826
- added J2: Conn_02x18_Odd_Even, Connector_Samtec_HLE_THT:Samtec_HLE-118-02-xx-DV-TE_2x18_P2.54mm_Horizontal, symbol Connector_Generic:Conn_02x18_Odd_Even
- added JP10, JP3: SolderJumper_2_Bridged, Jumper:SolderJumper-2_P1.3mm_Open_RoundedPad1.0x1.5mm, symbol Jumper:SolderJumper_2_Bridged
- added JP11, JP9: Jumper_2_Closed, Jumper:SolderJumper-2_P1.3mm_Bridged_RoundedPad1.0x1.5mm, symbol Jumper:Jumper_2_Open
- added JP2: SolderJumper_2_Bridged, Jumper:SolderJumper-2_P1.3mm_Bridged_RoundedPad1.0x1.5mm, symbol Jumper:SolderJumper_2_Bridged
- added JP4: Jumper_2_Open, Jumper:SolderJumper-2_P1.3mm_Open_RoundedPad1.0x1.5mm, symbol Jumper:Jumper_2_Open
- added R16: 180K, Resistor_SMD:R_0603_1608Metric, symbol Device:R
- added R20: 68K, Resistor_SMD:R_0603_1608Metric, symbol Device:R
- added R8: 4K7, Resistor_SMD:R_0603_1608Metric, symbol Device:R
- added R9: 1K, Resistor_SMD:R_0603_1608Metric, symbol Device:R
- added TP6, TP7, TP8, TP9: TestPoint, TestPoint:TestPoint_THTPad_D1.0mm_Drill0.5mm, symbol Connector:TestPoint
- added U4: MCP2562-E-SN, Package_SO:SOIC-8_3.9x4.9mm_P1.27mm, symbol Interface_CAN_LIN:MCP2562-E-SN
- added Y2: Crystal, Crystal:Crystal_SMD_3215-2Pin_3.2x1.5mm, symbol Device:Crystal
- C1: renamed from C6; footprint Resistor_SMD:R_0603_1608Metric -> Capacitor_SMD:C_0603_1608Metric; LCSC (none) -> C23630
- C10: renamed from C9; LCSC (none) -> C1634
- C11: renamed from C10; LCSC (none) -> C1634
- C2: renamed from C7; LCSC (none) -> C14663
- C3: renamed from C8; LCSC (none) -> C14663
- C4: renamed from C1; LCSC (none) -> C15850
- C5: renamed from C2; LCSC (none) -> C14663
- C6: renamed from C3; LCSC (none) -> C14663
- C7: renamed from C4; LCSC (none) -> C14663
- C8: renamed from C5; LCSC (none) -> C14663
- C9: renamed from C11; LCSC (none) -> C14663
- D1: LCSC (none) -> C2286
- FB1, FB2: footprint Resistor_SMD:R_0805_2012Metric -> Resistor_SMD:R_1206_3216Metric; LCSC (none) -> C94305
- P1: symbol Connector:USB_C_Receptacle_USB2.0 -> TeensyTest-rescue:USB_C_Receptacle_USB2.0-Connector; LCSC (none) -> C165948
- R1: renamed from R6; LCSC (none) -> C22935
- R2: renamed from R1; LCSC (none) -> C23186
- R3: renamed from R2; LCSC (none) -> C23186
- R4: renamed from R3; LCSC (none) -> C23140
- R5: renamed from R4; LCSC (none) -> C23140
- R6: renamed from R5; LCSC (none) -> C23179
- R7: LCSC (none) -> C23179
- U1: renamed from U3; footprint Package_DFN_QFN:QFN-16-1EP_3x3mm_P0.5mm_EP1.8x1.8mm -> Package_QFP:TQFP-32_7x7mm_P0.8mm; symbol MCU_NXP_Kinetis:MKL02Z32VFG4 -> MCU_NXP_Kinetis:MKL04Z32VLC4
- Y1: footprint Crystal:Crystal_SMD_Abracon_ABM3B-4Pin_5.0x3.2mm -> Crystal:Crystal_SMD_3225-4Pin_3.2x2.5mm; LCSC (none) -> C13738
- renumbered U2 to U3
Connections:
- net labels added: +12V, +5V, 14_A0, 15_A1, 2, 20_A6, 21_A7, 22_A8, 23_A9, 24, 26, 27, 29, 30, 31, 33, 5, 6, 8, 9, A10, A10_1, A11, A11_1, A12, A13, CANH, CANL, CRX, CTX, DAC_A14, D_N, D_P, GND1, IGN, LIN, Q_STBY, VCC, WDO
- net labels removed: DM, DP
- wire segments 91 -> 221
- no-connect marks 36 -> 8
Other:
- note added: "J1 Rotation:\n180???"
- note added: "Master mode by default."
- note added: "P1 Rotation:\n90 deg"
- note added: "Pins updated to swap them the right way round \nand STBY pin control added 03 March 2021"
- note added: "REMEMBER: find out a way of not supplying +5V to the regulator\nwhen powered by USB!\nDone by way of jumpers, I think...\nIMPORTANT - change pins on regulator. They are WRONG!"
- note added: "V2 for PWM - swapped 6 and D0"
- moved on the sheet: C4, C5, C6, C7, C8, C9, H1, H2
